File: Alexiares_LPF_RX_In.kicad_pcb (KiCad board)
At the start: 2 copper layers, 50 x 50 mm, 21 parts, among them J1 CONN_COAXIAL, J2 CONN_COAXIAL, J3 Conn_01x03, J5 CONN_COAXIAL

Commit message: Caps changed for ATC footprint
Parts:
- C10, C11, C12, C14, C8, C9: footprint Capacitors_SMD:C_1206_HandSoldering -> ATC_B:ATC_500_HandSoldering
- moved C10 8.86 mm to (114.5, 60.5), turned to 90 degrees
- moved C9 8.02 mm to (123.0, 69.5)
- moved C12 0.71 mm to (102.5, 69.5)
Routing:
- net Net-(C11-Pad1): track 20.4 -> 26.9 mm
- net Net-(C8-Pad1): track 16.4 -> 22.6 mm
- net Net-(C14-Pad1): track 20.4 -> 25.5 mm
- net Net-(C10-Pad1): track 23.8 -> 23.3 mm

Commit message: some via added
Routing:
- net GND: track 276.4 -> 301.2 mm, vias 71 -> 84
Changed lines of the file:
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@@
     (thickness 1.6)
     (drawings 9)
-    (tracks 225)
+    (tracks 257)
     (zones 0)
     (modules 21)
@@
   )
   (setup
-    (last_trace_width 1.6)
+    (last_trace_width 0.25)
     (user_trace_width 1.3)
     (user_trace_width 1.6)
@@
     (tags "capacitor ATC")
     (attr smd)
-    (fp_text reference C8 (at 0 4.064 90) (layer B.SilkS)
+    (fp_text reference C8 (at 4.485 0 180) (layer B.SilkS)
       (effects (font (size 1 1) (thickness 0.15)) (justify mirror))
     )
@@
     (tags "capacitor ATC")
     (attr smd)
-    (fp_text reference C9 (at 0 4.064 270) (layer B.SilkS)
+    (fp_text reference C9 (at 4.795 0.445 360) (layer B.SilkS)
       (effects (font (size 1 1) (thickness 0.15)) (justify mirror))
     )
@@
     (tags "capacitor ATC")
     (attr smd)
-    (fp_text reference C10 (at 0 4.064 90) (layer B.SilkS)
+    (fp_text reference C10 (at -4.905 -0.2 180) (layer B.SilkS)
       (effects (font (size 1 1) (thickness 0.15)) (justify mirror))
     )
@@
     (tags "capacitor ATC")
     (attr smd)
-    (fp_text reference C11 (at 0 4.064 90) (layer B.SilkS)
+    (fp_text reference C11 (at 4.485 -0.59 180) (layer B.SilkS)
       (effects (font (size 1 1) (thickness 0.15)) (justify mirror))
     )
@@
     (tags "capacitor ATC")
     (attr smd)
-    (fp_text reference C12 (at 0 4.064 270) (layer B.SilkS)
+    (fp_text reference C12 (at 4.16 -0.37 360) (layer B.SilkS)
       (effects (font (size 1 1) (thickness 0.15)) (justify mirror))
     )
@@
     (tags "capacitor ATC")
     (attr smd)
-    (fp_text reference C14 (at 0 4.064 270) (layer B.SilkS)
+    (fp_text reference C14 (at -5.12 -0.52 360) (layer B.SilkS)
       (effects (font (size 1 1) (thickness 0.15)) (justify mirror))
     )
@@
     )
   )
-  (gr_text "TXRX_RLY\n+12V\nGnd" (at 102.5 50) (layer B.SilkS)
+  (gr_text "TXRX_RLY\n\n+12V\n\nGnd" (at 102.87 49.53) (layer B.SilkS)
     (effects (font (size 1.5 1.5) (thickness 0.3)) (justify right mirror))
   )
@@
   (segment (start 101.0762 50) (end 104.46 50) (width 1.6) (layer F.Cu) (net 1))
   (segment (start 104.46 50) (end 106 51.54) (width 1.6) (layer F.Cu) (net 1))
+  (segment (start 112 37.46) (end 112 38.5) (width 0.25) (layer B.Cu) (net 2))
+  (segment (start 117.5 39) (end 119.04 37.46) (width 0.25) (layer B.Cu) (net 2) (status 800000))
+  (via (at 117.5 39) (size 0.6) (drill 0.4) (layers F.Cu B.Cu) (net 2))
+  (segment (start 116.5 40) (end 117.5 39) (width 0.25) (layer F.Cu) (net 2))
+  (via (at 116.5 40) (size 0.6) (drill 0.4) (layers F.Cu B.Cu) (net 2))
+  (segment (start 115.5 41) (end 116.5 40) (width 0.25) (layer B.Cu) (net 2))
+  (via (at 115.5 41) (size 0.6) (drill 0.4) (layers F.Cu B.Cu) (net 2))
+  (segment (start 114.5 41) (end 115.5 41) (width 0.25) (layer F.Cu) (net 2))
+  (via (at 114.5 41) (size 0.6) (drill 0.4) (layers F.Cu B.Cu) (net 2))
+  (segment (start 113.5 40) (end 114.5 41) (width 0.25) (layer B.Cu) (net 2))
+  (via (at 113.5 40) (size 0.6) (drill 0.4) (layers F.Cu B.Cu) (net 2))
+  (segment (start 112.5 39) (end 113.5 40) (width 0.25) (layer F.Cu) (net 2))
+  (via (at 112.5 39) (size 0.6) (drill 0.4) (layers F.Cu B.Cu) (net 2))
+  (segment (start 112 38.5) (end 112.5 39) (width 0.25) (layer B.Cu) (net 2))
+  (segment (start 119.04 37.46) (end 119.96 37.46) (width 0.25) (layer B.Cu) (net 2) (status C00000))
+  (segment (start 119 55) (end 119 53.5) (width 0.25) (layer F.Cu) (net 2))
+  (segment (start 118.5 44) (end 119.96 42.54) (width 0.25) (layer B.Cu) (net 2) (status 800000))
+  (via (at 118.5 44) (size 0.6) (drill 0.4) (layers F.Cu B.Cu) (net 2))
+  (segment (start 118.5 45.5) (end 118.5 44) (width 0.25) (layer F.Cu) (net 2))
+  (via (at 118.5 45.5) (size 0.6) (drill 0.4) (layers F.Cu B.Cu) (net 2))
+  (segment (start 118.5 47) (end 118.5 45.5) (width 0.25) (layer B.Cu) (net 2))
+  (via (at 118.5 47) (size 0.6) (drill 0.4) (layers F.Cu B.Cu) (net 2))
+  (segment (start 118.5 48.5) (end 118.5 47) (width 0.25) (layer F.Cu) (net 2))
+  (via (at 118.5 48.5) (size 0.6) (drill 0.4) (layers F.Cu B.Cu) (net 2))
+  (segment (start 118.5 50) (end 118.5 48.5) (width 0.25) (layer B.Cu) (net 2))
+  (via (at 118.5 50) (size 0.6) (drill 0.4) (layers F.Cu B.Cu) (net 2))
+  (segment (start 118.5 51.5) (end 118.5 50) (width 0.25) (layer F.Cu) (net 2))
+  (via (at 118.5 51.5) (size 0.6) (drill 0.4) (layers F.Cu B.Cu) (net 2))
+  (segment (start 118.5 53) (end 118.5 51.5) (width 0.25) (layer B.Cu) (net 2))
+  (via (at 118.5 53) (size 0.6) (drill 0.4) (layers F.Cu B.Cu) (net 2))
+  (segment (start 119 53.5) (end 118.5 53) (width 0.25) (layer F.Cu) (net 2))
   (segment (start 99.0762 54.54) (end 100.54 54.54) (width 0.25) (layer B.Cu) (net 2))
   (via (at 105.5 55) (size 0.6) (drill 0.4) (layers F.Cu B.Cu) (net 2))
@@
   (segment (start 129.96 37.46) (end 130 37.5) (width 0.25) (layer F.Cu) (net 2))
   (segment (start 132.5 40) (end 135 40) (width 0.25) (layer B.Cu) (net 2))
-  (segment (start 110.04 37.46) (end 114.96 37.46) (width 0.25) (layer B.Cu) (net 2))
+  (segment (start 110.04 37.46) (end 112 37.46) (width 0.25) (layer B.Cu) (net 2))
+  (segment (start 112 37.46) (end 114.96 37.46) (width 0.25) (layer B.Cu) (net 2))
   (segment (start 115.04 37.46) (end 119.96 37.46) (width 0.25) (layer F.Cu) (net 2))
   (segment (start 115 37.5) (end 115.04 37.46) (width 0.25) (layer F.Cu) (net 2))

Commit message: DEPRECATED PROJECT, DO NOT USE WITH ALEX
Parts:
- added J4: CONN_COAXIAL, SMA_PINS:SMA_EDGE_NRW, F.Cu at (116.0, 82.2)
- added J6: CONN_COAXIAL, SMA_PINS:SMA_EDGE_NRW, F.Cu at (122.5, 37.7)
- added J7: CONN_COAXIAL, SMA_PINS:SMA_EDGE_NRW, F.Cu at (107.5, 37.4)
- moved C9 16.8 mm to (133.2, 56.2), turned to 90 degrees
- moved C11 9.22 mm to (112.0, 68.0), turned to 0 degrees
- moved C8 8.29 mm to (133.2, 66.5), turned to 270 degrees
- moved C10 1.61 mm to (116.1, 60.7)
- moved L4 0.10 mm to (119.9, 64.0), turned to 270 degrees
- turned L1 to 90 degrees
Routing:
- net GND: track 301.2 -> 351.5 mm, vias 84 -> 119
- net Net-(C8-Pad2): track 36.5 -> 29.3 mm
- net Net-(C10-Pad1): track 23.3 -> 18.6 mm
- net Net-(J5-Pad1): track 16.2 -> 20.8 mm
- net Net-(C8-Pad1): track 22.6 -> 19.0 mm
- net Net-(J2-Pad1): track 16.2 -> 18.7 mm
- net Net-(C11-Pad1): track 26.9 -> 28.0 mm
Other:
- board text added: "THIS PROJECT IS DEPRECATED DO NOT USE"
- board text added: "design f6itu"
- board text added: "Ἀλεξιάρης to Alexiares HPF"
- board text removed: "Alex HPF"
